File: pcb/drivers.kicad_sch (KiCad schematic)
At the start: 38 parts, among them J1 DRV_ICSP, P3 CARRIAGE_STEPPER, P4 DRIVE_MOTOR, P5 LF_SOLENOID, Q1 IRLR110TRPBF, Q2 IRLR110TRPBF, Q3 IRLR110TRPBF, Q4 IRLR110TRPBF, U2 ATtiny404-SS

Commit message: Tweak PSU
Parts:
- renumbered C3 to C12, C4 to C13, C5 to C14, C6 to C15, C7 to C16, C8 to C17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
