File: pcb/micro.kicad_sch (KiCad schematic)
At the start: 47 parts, among them J3 ICSP, J4 KB_COL, J5 CASE_OPEN, J6 KB_ROW, J7 I2C_TST, Q5 T2N7002AK, U4 ATmega328P-MM, U5 TCA9534, U6 23LC1024, U7 47C04, U8 TCA9534

Commit message: Tweak PSU
Parts:
- renumbered C16 to C1, C25 to C10, C26 to C11, C17 to C2, C18 to C3, C19 to C4, C20 to C5, C21 to C6, C22 to C7, C23 to C8, C24 to C9, D6 to D1, D7 to D2, D8 to D3, D9 to D4, J3 to J1, J4 to J2, J5 to J3, J6 to J4, J7 to J5, NT3 to NT1, Q5 to Q1, R10 to R1, R19 to R10, R20 to R11, R21 to R12, R22 to R13, R23 to R14, R24 to R15, R25 to R16, R26 to R17, R27 to R18, R28 to R19, R11 to R2, R12 to R3, R13 to R4, R14 to R5, R15 to R6, R16 to R7, R17 to R8, R18 to R9, U4 to U1, U5 to U2, U6 to U3, U7 to U4, U8 to U5

Commit message: Rename kicad project
Parts:
- U3: symbol typerwriter:23LC1024 -> retrotype:23LC1024
Changed lines of the file:
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@@
     (company "Zach Anderson")
   )
-  (bus_alias "I2C" (members "SCL" "SDA"))
   (bus_alias "RS232" (members "TX" "DTR" "RTS" "RX" "CTS" "DSR" "RI" "DCD"))
   (bus_alias "STEPPERS" (members "DAISY_WHEEL_STEPPER_STEP" "CARRIAGE_STEPPER_STEP"))
+  (bus_alias "I2C" (members "SCL" "SDA"))
   (junction (at 207.01 74.93) (diameter 0) (color 0 0 0 0)
   )
@@
     (pin "1")
   )
-  (symbol (lib_id "typerwriter:23LC1024") (at 135.89 36.83 0) (unit 1)
+  (symbol (lib_id "retrotype:23LC1024") (at 135.89 36.83 0) (unit 1)
     (in_bom yes) (on_board yes)
     (property "Reference" "U3" (id 0) (at 143.51 27.94 0))
