File: pcb/rs232.kicad_sch (KiCad schematic)
At the start: 9 parts, among them J2 DB9_Male

Commit message: Tweak PSU
Parts:
- gave numbers to parts that had none: 7
- renumbered C12 to C21, J2 to J7
Connections:
- no-connect marks 4 -> 2
Changed lines of the file:
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@@
   (junction (at 163.83 109.22) (diameter 0) (color 0 0 0 0)
   )
-  (no_connect (at -82.55 171.45))
   (no_connect (at 110.49 124.46))
   (no_connect (at 110.49 92.71))
-  (no_connect (at -82.55 161.29))
   (bus_entry (at 91.44 24.13) (size -2.54 2.54)
     (stroke (width 0) (type default) (color 0 0 0 0))
@@
     (stroke (width 0) (type default) (color 0 0 0 0))
   )
-  (wire (pts (xy -87.63 156.21) (xy -82.55 156.21))
-    (stroke (width 0) (type default) (color 0 0 0 0))
-  )
   (bus (pts (xy 88.9 34.29) (xy 88.9 36.83))
     (stroke (width 0) (type default) (color 0 0 0 0))
@@
   )
   (wire (pts (xy 163.83 119.38) (xy 163.83 120.65))
-    (stroke (width 0) (type default) (color 0 0 0 0))
-  )
-  (wire (pts (xy -87.63 166.37) (xy -82.55 166.37))
     (stroke (width 0) (type default) (color 0 0 0 0))
   )
@@
     (effects (font (size 1.27 1.27)) (justify left bottom))
   )
-  (label "RX" (at -87.63 166.37 0)
-    (effects (font (size 1.27 1.27)) (justify left bottom))
-  )
   (label "DCD" (at 105.41 114.3 0)
     (effects (font (size 1.27 1.27)) (justify left bottom))
@@
   (label "L_CTS" (at 157.48 129.54 180)
     (effects (font (size 1.27 1.27)) (justify right bottom))
-  )
-  (label "TX" (at -87.63 156.21 0)
-    (effects (font (size 1.27 1.27)) (justify left bottom))
   )
   (label "DSR" (at 99.06 41.91 180)
@@
   (symbol (lib_id "Connector:DB9_Male") (at 193.04 35.56 0) (mirror x) (unit 1)
     (in_bom yes) (on_board yes)
-    (property "Reference" "J2" (id 0) (at 190.9572 17.9832 0))
+    (property "Reference" "J7" (id 0) (at 190.9572 17.9832 0))
     (property "Value" "DB9_Male" (id 1) (at 190.9572 20.2946 0))
     (property "Footprint" "" (id 2) (at 193.04 35.56 0)
@@
   (symbol (lib_id "power:VCC") (at 130.81 62.23 0) (unit 1)
     (in_bom yes) (on_board yes)
-    (property "Reference" "#PWR037" (id 0) (at 130.81 66.04 0)
+    (property "Reference" "#PWR085" (id 0) (at 130.81 66.04 0)
       (effects (font (size 1.27 1.27)) hide)
     )
@@
     (pin "1")
   )
-  (symbol (lib_id "power:GND") (at -62.23 184.15 0) (unit 1)
-    (in_bom yes) (on_board yes)
-    (property "Reference" "#PWR038" (id 0) (at -62.23 190.5 0)
-      (effects (font (size 1.27 1.27)) hide)
-    )
-    (property "Value" "GND" (id 1) (at -62.103 188.5442 0))
-    (property "Footprint" "" (id 2) (at -62.23 184.15 0)
-      (effects (font (size 1.27 1.27)) hide)
-    )
-    (property "Datasheet" "" (id 3) (at -62.23 184.15 0)
-      (effects (font (size 1.27 1.27)) hide)
-    )
-    (pin "1")
-  )
   (symbol (lib_id "Device:C") (at 135.89 63.5 270) (unit 1)
     (in_bom yes) (on_board yes)
-    (property "Reference" "C12" (id 0) (at 135.89 57.0992 90))
+    (property "Reference" "C21" (id 0) (at 135.89 57.0992 90))
     (property "Value" "100n" (id 1) (at 135.89 59.4106 90))
     (property "Footprint" "" (id 2) (at 132.08 64.4652 0)
@@
   (symbol (lib_id "power:GND") (at 139.7 63.5 90) (unit 1)
     (in_bom yes) (on_board yes)
-    (property "Reference" "#PWR039" (id 0) (at 146.05 63.5 0)
+    (property "Reference" "#PWR087" (id 0) (at 146.05 63.5 0)
       (effects (font (size 1.27 1.27)) hide)
     )
@@
   (symbol (lib_id "power:GND") (at 165.1 85.09 90) (unit 1)
     (in_bom yes) (on_board yes)
-    (property "Reference" "#PWR040" (id 0) (at 171.45 85.09 0)
+    (property "Reference" "#PWR088" (id 0) (at 171.45 85.09 0)
       (effects (font (size 1.27 1.27)) hide)
     )
@@
   (symbol (lib_id "power:GND") (at 185.42 45.72 270) (unit 1)
     (in_bom yes) (on_board yes)
-    (property "Reference" "#PWR041" (id 0) (at 179.07 45.72 0)
+    (property "Reference" "#PWR090" (id 0) (at 179.07 45.72 0)
       (effects (font (size 1.27 1.27)) hide)
     )
@@
   (symbol (lib_id "Device:C") (at 153.67 76.2 0) (unit 1)
     (in_bom yes) (on_board yes) (fields_autoplaced)
-    (property "Reference" "C?" (id 0) (at 156.591 75.3653 0)
+    (property "Reference" "C22" (id 0) (at 156.591 75.3653 0)
       (effects (font (size 1.27 1.27)) (justify left))
     )
@@
   (symbol (lib_id "power:GND") (at 130.81 152.4 0) (unit 1)
     (in_bom yes) (on_board yes) (fields_autoplaced)
-    (property "Reference" "#PWR?" (id 0) (at 130.81 158.75 0)
+    (property "Reference" "#PWR086" (id 0) (at 130.81 158.75 0)
       (effects (font (size 1.27 1.27)) hide)
     )
@@
   (symbol (lib_id "typerwriter:MAX3243") (at 130.81 111.76 0) (unit 1)
     (in_bom yes) (on_board yes)
-    (property "Reference" "U?" (id 0) (at 116.84 68.58 0)
+    (property "Reference" "U7" (id 0) (at 116.84 68.58 0)
       (effects (font (size 1.27 1.27)) (justify left))
     )
@@
   (symbol (lib_id "Device:R") (at 163.83 115.57 0) (unit 1)
     (in_bom yes) (on_board yes) (fields_autoplaced)
-    (property "Reference" "R?" (id 0) (at 165.608 114.7353 0)
+    (property "Reference" "R29" (id 0) (at 165.608 114.7353 0)
       (effects (font (size 1.27 1.27)) (justify left))
     )
@@
   (symbol (lib_id "Device:C") (at 171.45 115.57 0) (unit 1)
     (in_bom yes) (on_board yes) (fields_autoplaced)
-    (property "Reference" "C?" (id 0) (at 174.371 114.7353 0)
+    (property "Reference" "C25" (id 0) (at 174.371 114.7353 0)
       (effects (font (size 1.27 1.27)) (justify left))
     )
@@
   (symbol (lib_id "power:GND") (at 167.64 121.92 0) (unit 1)
     (in_bom yes) (on_board yes) (fields_autoplaced)
-    (property "Reference" "#PWR?" (id 0) (at 167.64 128.27 0)
+    (property "Reference" "#PWR089" (id 0) (at 167.64 128.27 0)
       (effects (font (size 1.27 1.27)) hide)
     )
@@
   (symbol (lib_id "power:VCC") (at 87.63 49.53 270) (unit 1)
     (in_bom yes) (on_board yes) (fields_autoplaced)
-    (property "Reference" "#PWR?" (id 0) (at 83.82 49.53 0)
+    (property "Reference" "#PWR082" (id 0) (at 83.82 49.53 0)
       (effects (font (size 1.27 1.27)) hide)
     )
@@
   (symbol (lib_id "power:GND") (at 110.49 85.09 270) (unit 1)
     (in_bom yes) (on_board yes) (fields_autoplaced)
-    (property "Reference" "#PWR?" (id 0) (at 104.14 85.09 0)
+    (property "Reference" "#PWR083" (id 0) (at 104.14 85.09 0)
       (effects (font (size 1.27 1.27)) hide)
     )
@@
   (symbol (lib_id "Device:C") (at 106.68 76.2 0) (unit 1)
     (in_bom yes) (on_board yes)
-    (property "Reference" "C?" (id 0) (at 106.68 73.66 0)
+    (property "Reference" "C20" (id 0) (at 106.68 73.66 0)
       (effects (font (size 1.27 1.27)) (justify left))
     )
@@
   (symbol (lib_id "Device:C") (at 154.94 92.71 90) (unit 1)
     (in_bom yes) (on_board yes)
-    (property "Reference" "C?" (id 0) (at 152.4 91.44 90))
+    (property "Reference" "C24" (id 0) (at 152.4 91.44 90))
     (property "Value" "330n" (id 1) (at 151.13 93.98 90))
     (property "Footprint" "" (id 2) (at 158.75 91.7448 0)
@@
   (symbol (lib_id "Device:C") (at 154.94 85.09 90) (unit 1)
     (in_bom yes) (on_board yes)
-    (property "Reference" "C?" (id 0) (at 152.4 83.82 90))
+    (property "Reference" "C23" (id 0) (at 152.4 83.82 90))
     (property "Value" "330n" (id 1) (at 151.13 86.36 90))
     (property "Footprint" "" (id 2) (at 158.75 84.1248 0)
@@
   (symbol (lib_id "power:VCC") (at 110.49 88.9 90) (unit 1)
     (in_bom yes) (on_board yes) (fields_autoplaced)
-    (property "Reference" "#PWR?" (id 0) (at 114.3 88.9 0)
-      (effects (font (size 1.27 1.27)) hide)
-    )
+    (property "Reference" "#PWR084" (id 0) (at 114.3 88.9 0)
+      (effects (font (size 1.27 1.27)) hide)
+    )

Commit message: Rename kicad project
Parts:
- U7: symbol typerwriter:MAX3243 -> retrotype:MAX3243
Changed lines of the file:
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@@
     (pin "1")
   )
-  (symbol (lib_id "typerwriter:MAX3243") (at 130.81 111.76 0) (unit 1)
+  (symbol (lib_id "retrotype:MAX3243") (at 130.81 111.76 0) (unit 1)
     (in_bom yes) (on_board yes)
     (property "Reference" "U7" (id 0) (at 116.84 68.58 0)
